Commit message: Fix undefined parameters min_angle, max_angle in urdf macros sick_tim_5xx and sick_mrs_1xxx

File: urdf/sick_scan.urdf.xacro (robot description, xacro)
@@ -4,8 +4,9 @@
   xmlns:sensor="http://playerstage.sourceforge.net/gazebo/xmlschema/#sensor"
   xmlns:xacro="http://ros.org/wiki/xacro">
-  <xacro:macro name="sick_tim_5xx" params="name ros_topic">
+  <xacro:macro name="sick_tim_5xx" params="name ros_topic min_angle:=-2.357 max_angle:=2.357 samples:=271">
     <xacro:sick_tim name="${name}" ros_topic="${ros_topic}"
       length="0.06" width="0.06" height="0.079" mass="0.150" z_offset="0.05595"
-      min_range="0.05" max_range="4.0" samples="271"
+      min_angle="${min_angle}" max_angle="${max_angle}"
+      min_range="0.05" max_range="4.0" samples="${samples}"
       mesh="package://sick_scan/meshes/sick_tim_5xx.stl" />
   </xacro:macro>
@@ -24,8 +25,9 @@
       mesh="package://sick_scan/meshes/sick_tim_5xx.stl" />
   </xacro:macro>
-  <xacro:macro name="sick_mrs_1xxx" params="name ros_topic">
+  <xacro:macro name="sick_mrs_1xxx" params="name ros_topic min_angle:=-2.357 max_angle:=2.357 samples:=271">
     <xacro:sick_tim name="${name}" ros_topic="${ros_topic}"
       length="0.06" width="0.06" height="0.079" mass="0.150" z_offset="0.05595"
-      min_range="0.05" max_range="4.0" samples="271"
+      min_angle="${min_angle}" max_angle="${max_angle}"
+      min_range="0.05" max_range="4.0" samples="${samples}"
       mesh="package://sick_scan/meshes/sick_tim_5xx.stl" />
   </xacro:macro>
